File: Hardware/schematic.sch (EAGLE design)
At the start: 105 parts, among them IC1 BQ25180YBGR, IC2 DRV2605YZFR, IC3 BMA423, IC9 RT6160AWSC, J1 503480-2400, J2 TC2030-IDC, J4 KH-TYPE-C-16P, Q3 SI1308EDL-T1-GE3, U1 NRF52840_QF, U3 MAX17048G+T10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

Commit message: done
Parts:
- EPD_C9: device InkTime_v5:PERFECT_0402_CAP_0402 -> new_InkTime_v5:PERFECT_0402_CAP_0402
